Commit message: chore

File: robots/go1l2_description/xacro/gazebo.xacro (robot description, xacro)
@@ -17,4 +17,18 @@
                 <material>Gazebo/Yellow</material>
             </plot>
+        </plugin>
+    </gazebo>
+    <!-- Show the accurate position of trunk center. -->
+    <gazebo>
+        <plugin filename="libgazebo_ros_p3d.so" name="gazebo_ros_p3d">
+            <frameName>world</frameName>           <!-- 父坐标系 -->
+            <robotNamespace>/</robotNamespace>
+            <bodyName>base</bodyName>         <!-- 子坐标系（机器人底盘） -->
+            <topicName>ground_truth</topicName>
+            <xyzOffsets>0 0 0</xyzOffsets>
+            <rpyOffsets>0 0 0</rpyOffsets>
+            <gaussianNoise>0</gaussianNoise>
+            <alwaysOn>true</alwaysOn>
+            <updateRate>250.0</updateRate>
         </plugin>
     </gazebo>

File: robots/go1l2_description/xacro/leg.xacro (robot description, xacro)
@@ -124,5 +124,5 @@
                     </xacro:if>
                 </geometry>
-                <!-- <material name="orange"/> -->
+                <material name="orange"/>
             </visual>
             <collision>
@@ -183,5 +183,5 @@
                     <mesh filename="package://go1l2_description/meshes/calf.dae" scale="1 1 1"/>
                 </geometry>
-                <!-- <material name="orange"/> -->
+                <material name="orange"/>
             </visual>
             <collision>
@@ -234,5 +234,5 @@
                     <sphere radius="${foot_radius-0.01}"/>
                 </geometry>
-                <!-- <material name="orange"/> -->
+                <material name="orange"/>
             </visual>
             <collision>

File: robots/go1l2_description/xacro/robot.xacro (robot description, xacro)
@@ -2,11 +2,15 @@
 <robot name="go1l2" xmlns:xacro="http://www.ros.org/wiki/xacro">
     <xacro:arg name="DEBUG" default="false"/>
+    <!-- TODO: 将深度相机和超声传感器隔离至单独的文件夹 -->
+    <!-- TODO: 添加不同种类的传感器包-->
+    <!-- TODO: 给机器人的腿换一下不同的颜色 -->
+    <!-- TODO: 把机器人一开始就是卧倒的姿态，然后处于gazebo的(0， 0)处的位置 -->
+    <xacro:include filename="$(find go1l2_description)/xacro/colors.xacro"/>
     <xacro:include filename="$(find go1l2_description)/xacro/const.xacro"/>
-    <xacro:include filename="$(find go1l2_description)/xacro/materials.xacro"/>
     <xacro:include filename="$(find go1l2_description)/xacro/leg.xacro"/>
-    <!-- <xacro:include filename="$(find go1l2_description)/xacro/stairs.xacro"/> -->
     <xacro:include filename="$(find go1l2_description)/xacro/gazebo.xacro"/>
     <xacro:include filename="$(find go1l2_description)/xacro/depthCamera.xacro"/>
     <xacro:include filename="$(find go1l2_description)/xacro/ultraSound.xacro"/>
+    <!-- <xacro:include filename="$(find go1l2_description)/xacro/stairs.xacro"/> -->
     <!-- <xacro:include filename="$(find go1l2_gazebo)/launch/stairs.urdf.xacro"/> -->
     <!-- <xacro:stairs stairs="15" xpos="0" ypos="0" zpos="0" /> -->
@@ -14,4 +18,5 @@
     <!-- Actually, the rotor will rotate and the joint is not fixed. Reduction ratio should be considered. -->
     <!-- Debug mode will hung up the robot, use "true" or "false" to switch it. -->
+    <!-- DEBUG模式将会把机器人悬挂起来 -->
     <xacro:if value="$(arg DEBUG)">
         <link name="world"/>
@@ -39,7 +44,9 @@
             <origin rpy="0 0 0" xyz="0 0 0"/>
             <geometry>
-                <mesh filename="package://go1l2_description/meshes/trunk.dae" scale="1 1 1"/>
+                <mesh filename="package://go1l2_description/meshes/trunk.stl" scale="1 1 1"/>
             </geometry>
-            <!-- <material name="orange"/> -->
+            <material name="orange">
+                <color rgba="1.0 0.4235 0.0392 1.0"/>
+            </material>
         </visual>
         <collision>
