Commit message: add lidar for dog

File: robots/go1l2_description/xacro/robot.xacro (robot description, xacro)
@@ -94,4 +94,13 @@
     <xacro:leg name="RR" mirror="-1" mirror_dae="False"  front_hind="-1" front_hind_dae="False" />
     <xacro:leg name="RL" mirror="1"  mirror_dae="True"   front_hind="-1" front_hind_dae="False" />
+    <xacro:arg name="gpu" default="false"/>
+    <xacro:property name="gpu" value="$(arg gpu)" />
+    <xacro:property name="lidar_frame_name" value="BPearl_Lidar"/>
+    <xacro:arg name="organize_cloud" default="false"/>
+    <xacro:property name="organize_cloud" value="$(arg organize_cloud)" />
+    <xacro:include filename="$(find gazebo_sensors)/lidars/RS-BPearl/xacro/RS-BPearl.xacro"/>
+    <xacro:RS-BPearl parent="trunk" name="${lidar_frame_name}" topic="/bpearl_points" organize_cloud="${organize_cloud}" hz="15" samples="1000" gpu="${gpu}">
+        <origin xyz="0.30 0.0 0.0" rpy="0 1.5708 0" />
+    </xacro:RS-BPearl>
     <xacro:depthCamera camID="1" name="face">
         <origin rpy="${PI} 0 0" xyz="0.2785 0.0125 0.0167"/>

Commit message: update robot.xacro for lidar

File: robots/go1l2_description/xacro/robot.xacro (robot description, xacro)
@@ -94,5 +94,29 @@
     <xacro:leg name="RR" mirror="-1" mirror_dae="False"  front_hind="-1" front_hind_dae="False" />
     <xacro:leg name="RL" mirror="1"  mirror_dae="True"   front_hind="-1" front_hind_dae="False" />
-    <xacro:arg name="gpu" default="false"/>
+    <!-- <joint name="lidar_joint" type="fixed">
+        <parent link="trunk"/>
+        <child link="lidar_link"/>
+        <origin rpy="0 0 0" xyz="0.0 0.0 0.15"/>
+    </joint>
+    <link name="imu_link">
+        <inertial>
+            <mass value="0.001"/>
+            <origin rpy="0 0 0" xyz="0 0 0"/>
+            <inertia ixx="0.0001" ixy="0" ixz="0" iyy="0.0001" iyz="0" izz="0.0001"/>
+        </inertial>
+        <visual>
+            <origin rpy="0 0 0" xyz="0 0 0"/>
+            <geometry>
+                <box size="0.001 0.001 0.001"/>
+            </geometry>
+        </visual>
+        <collision>
+            <origin rpy="0 0 0" xyz="0 0 0"/>
+            <geometry>
+                <box size=".001 .001 .001"/>
+            </geometry>
+        </collision>
+    </link> -->
+    <!-- <xacro:arg name="gpu" default="false"/>
     <xacro:property name="gpu" value="$(arg gpu)" />
     <xacro:property name="lidar_frame_name" value="BPearl_Lidar"/>
@@ -102,5 +126,12 @@
     <xacro:RS-BPearl parent="trunk" name="${lidar_frame_name}" topic="/bpearl_points" organize_cloud="${organize_cloud}" hz="15" samples="1000" gpu="${gpu}">
         <origin xyz="0.30 0.0 0.0" rpy="0 1.5708 0" />
-    </xacro:RS-BPearl>
+    </xacro:RS-BPearl> -->
+    <xacro:arg name="gpu" default="true"/>
+    <xacro:property name="gpu" value="$(arg gpu)" />
+    <xacro:property name="lidar_frame_name" value="VLP-16"/>
+    <xacro:include filename="$(find gazebo_sensors)/lidars/VLP-16/xacro/VLP-16.xacro"/>
+    <xacro:VLP-16 parent="base" name="${lidar_frame_name}" topic="/vlp16_points" hz="10" samples="1000" gpu="${gpu}">
+        <origin xyz="0.0 0.0 0.15" rpy="0 0 0" />
+    </xacro:VLP-16>
     <xacro:depthCamera camID="1" name="face">
         <origin rpy="${PI} 0 0" xyz="0.2785 0.0125 0.0167"/>

Commit message: update go1l2 xacro, minus unused depth camera

File: robots/go1l2_description/xacro/robot.xacro (robot description, xacro)
@@ -134,5 +134,5 @@
         <origin xyz="0.0 0.0 0.15" rpy="0 0 0" />
     </xacro:VLP-16>
-    <xacro:depthCamera camID="1" name="face">
+    <!-- <xacro:depthCamera camID="1" name="face">
         <origin rpy="${PI} 0 0" xyz="0.2785 0.0125 0.0167"/>
     </xacro:depthCamera>
@@ -148,6 +148,6 @@
     <xacro:depthCamera camID="5" name="rearDown">
         <origin rpy="${PI} ${PI/2} 0" xyz="-0.0825 0.0125 -0.04365"/>
-    </xacro:depthCamera>
-    <joint name="camera_laserscan_joint_left" type="fixed">
+    </xacro:depthCamera> -->
+    <!-- <joint name="camera_laserscan_joint_left" type="fixed">
         <origin rpy="0 0.2618 0" xyz="0 0 0"/>
         <parent link="camera_left"/>
@@ -162,5 +162,5 @@
     </joint>
     <link name="camera_laserscan_link_right">
-    </link>
+    </link> -->
     <xacro:ultraSound name="left">
         <origin rpy="0 0.2618 ${PI/2}" xyz="-0.0535  0.0826 0.00868"/>

Commit message: update robot.xacro

File: robots/go1l2_description/xacro/robot.xacro (robot description, xacro)
@@ -132,5 +132,5 @@
     <xacro:include filename="$(find gazebo_sensors)/lidars/VLP-16/xacro/VLP-16.xacro"/>
     <xacro:VLP-16 parent="base" name="${lidar_frame_name}" topic="/vlp16_points" hz="10" samples="1000" gpu="${gpu}">
-        <origin xyz="0.0 0.0 0.15" rpy="0 0 0" />
+        <origin xyz="0.0 0.0 0.05" rpy="0 0 0" />
     </xacro:VLP-16>
     <!-- <xacro:depthCamera camID="1" name="face">

Commit message: fix: 原来的lidar侵入到go1身体里，导致没有controller加载的时候模型乱动，现在好了，不加载controller模型也不乱动了

File: robots/go1l2_description/xacro/robot.xacro (robot description, xacro)
@@ -132,5 +132,5 @@
     <xacro:include filename="$(find gazebo_sensors)/lidars/VLP-16/xacro/VLP-16.xacro"/>
     <xacro:VLP-16 parent="base" name="${lidar_frame_name}" topic="/vlp16_points" hz="10" samples="1000" gpu="${gpu}">
-        <origin xyz="0.0 0.0 0.05" rpy="0 0 0" />
+        <origin xyz="0.0 0.0 0.0575" rpy="0 0 0" />
     </xacro:VLP-16>
     <!-- <xacro:depthCamera camID="1" name="face">
