Commit message: feat: filp the face camera of go1l2

File: robots/go1l2_description/xacro/depthCamera.xacro (robot description, xacro)
@@ -40,11 +40,11 @@
                     <horizontal_fov>2.094</horizontal_fov>
                     <image>
-                        <width>928</width>
-                        <height>800</height>
+                        <width>1920</width>
+                        <height>1080</height>
                         <format>R8G8B8</format>
                     </image>
                     <clip>
                         <near>0.1</near>
-                        <far>5</far>
+                        <far>50</far>
                     </clip>
                 </camera>
@@ -62,5 +62,5 @@
                     <frameName>camera_optical_${name}</frameName>
                     <pointCloudCutoff>0.1</pointCloudCutoff>
-                    <pointCloudCutoffMax>1.5</pointCloudCutoffMax>
+                    <pointCloudCutoffMax>50</pointCloudCutoffMax>
                     <distortionK1>0.0</distortionK1>
                     <distortionK2>0.0</distortionK2>

File: robots/go1l2_description/xacro/robot.xacro (robot description, xacro)
@@ -1,4 +1,5 @@
 <?xml version="1.0"?>
-<robot name="go1l2" xmlns:xacro="http://www.ros.org/wiki/xacro">
+<robot name="go1l2"
+    xmlns:xacro="http://www.ros.org/wiki/xacro">
     <xacro:arg name="DEBUG" default="false"/>
     <!-- TODO: 将深度相机和超声传感器隔离至单独的文件夹 -->
@@ -59,8 +60,5 @@
             <origin rpy="0 0 0" xyz="${trunk_com_x} ${trunk_com_y} ${trunk_com_z}"/>
             <mass value="${trunk_mass}"/>
-            <inertia
-                ixx="${trunk_ixx}" ixy="${trunk_ixy}" ixz="${trunk_ixz}"
-                iyy="${trunk_iyy}" iyz="${trunk_iyz}"
-                izz="${trunk_izz}"/>
+            <inertia ixx="${trunk_ixx}" ixy="${trunk_ixy}" ixz="${trunk_ixz}" iyy="${trunk_iyy}" iyz="${trunk_iyz}" izz="${trunk_izz}"/>
         </inertial>
     </link>
@@ -90,8 +88,8 @@
         </collision>
     </link>
-    <xacro:leg name="FR" mirror="-1" mirror_dae= "False" front_hind="1"  front_hind_dae="True"  />
-    <xacro:leg name="FL" mirror="1"  mirror_dae="True"   front_hind="1"  front_hind_dae="True"  />
-    <xacro:leg name="RR" mirror="-1" mirror_dae="False"  front_hind="-1" front_hind_dae="False" />
-    <xacro:leg name="RL" mirror="1"  mirror_dae="True"   front_hind="-1" front_hind_dae="False" />
+    <xacro:leg name="FR" mirror="-1" mirror_dae= "False" front_hind="1" front_hind_dae="True" />
+    <xacro:leg name="FL" mirror="1" mirror_dae="True" front_hind="1" front_hind_dae="True" />
+    <xacro:leg name="RR" mirror="-1" mirror_dae="False" front_hind="-1" front_hind_dae="False" />
+    <xacro:leg name="RL" mirror="1" mirror_dae="True" front_hind="-1" front_hind_dae="False" />
     <!-- <joint name="lidar_joint" type="fixed">
         <parent link="trunk"/>
@@ -134,4 +132,7 @@
         <origin xyz="0.0 0.0 0.0575" rpy="0 0 0" />
     </xacro:VLP-16>
+    <xacro:depthCamera camID="1" name="face">
+        <origin rpy="0 0 0" xyz="0.2785 0.0125 0.0167"/>
+    </xacro:depthCamera>
     <!-- <xacro:depthCamera camID="1" name="face">
         <origin rpy="${PI} 0 0" xyz="0.2785 0.0125 0.0167"/>

Commit message: feat: update simulation camera rgb param

File: robots/go1l2_description/xacro/depthCamera.xacro (robot description, xacro)
@@ -9,19 +9,19 @@
         <link name="camera_${name}">
             <collision>
-            <origin xyz="0 0 0" rpy="0 0 0"/>
-            <geometry>
-                <box size=".001 .001 .001"/>
-            </geometry>
+                <origin xyz="0 0 0" rpy="0 0 0"/>
+                <geometry>
+                    <box size=".001 .001 .001"/>
+                </geometry>
             </collision>
             <visual>
-            <origin xyz="0 0 0" rpy="0 0 0"/>
-            <geometry>
-                <mesh filename="package://go1l2_description/meshes/depthCamera.dae" scale="1 1 1"/>
-            </geometry>
+                <origin xyz="0 0 0" rpy="0 0 0"/>
+                <geometry>
+                    <mesh filename="package://go1l2_description/meshes/depthCamera.dae" scale="1 1 1"/>
+                </geometry>
             </visual>
             <inertial>
-            <mass value="1e-5" />
-            <origin xyz="0 0 0" rpy="0 0 0"/>
-            <inertia ixx="1e-6" ixy="0" ixz="0" iyy="1e-6" iyz="0" izz="1e-6" />
+                <mass value="1e-5" />
+                <origin xyz="0 0 0" rpy="0 0 0"/>
+                <inertia ixx="1e-6" ixy="0" ixz="0" iyy="1e-6" iyz="0" izz="1e-6" />
             </inertial>
         </link>
@@ -46,5 +46,5 @@
                     <clip>
                         <near>0.1</near>
-                        <far>50</far>
+                        <far>5000</far>
                     </clip>
                 </camera>
